Commit message: Update turtlebot3_burger.urdf.xacro

File: turtlebot3_description/urdf/turtlebot3_burger.urdf.xacro (robot description, xacro)
@@ -140,3 +140,18 @@
     </inertial>
   </link>
+  <!--camera-->
+  <joint name="camera_joint" type="fixed">
+    <parent link="base_link"/>
+    <child link="camera_link"/>
+    <origin xyz="0.05 0 0.085" rpy="0 0 0"/>
+  </joint>
+  <link name="camera_link">
+    <visual>
+      <origin xyz="0 0 0.0" rpy="0 0 0"/>
+      <geometry>
+        <box size="0.02 0.05 0.03"/>
+      </geometry>>
+      <!-- <material name="Green" /> -->
+    </visual>>
+  </link>
 </robot>
