Commit message: fix camera_frame

File: turtlebot3_description/urdf/turtlebot3_burger.gazebo.xacro (robot description, xacro)
@@ -131,4 +131,5 @@
       <visualize>$(arg camera_visual)</visualize>
       <camera>
+          <!-- <pose>0 0 0 0 0 0</pose> -->
           <horizontal_fov>2.09</horizontal_fov>
           <image>
@@ -146,5 +147,5 @@
         <updateRate>30.0</updateRate>
         <cameraName>camera</cameraName>
-        <frameName>camera_link</frameName>
+        <frameName>camera_tf_link</frameName>
         <imageTopicName>/image_raw</imageTopicName>
         <cameraInfoTopicName>/camera_info</cameraInfoTopicName>

File: turtlebot3_description/urdf/turtlebot3_burger.urdf.xacro (robot description, xacro)
@@ -152,6 +152,25 @@
         <box size="0.02 0.05 0.03"/>
       </geometry>>
-      <!-- <material name="Green" /> -->
     </visual>>
   </link>
+  <!-- <joint name="camera_joint" type="fixed">
+    <parent link="base_link"/>
+    <child link="camera_link"/>
+    <origin xyz="0.05 0 0.085" rpy="-1.57 0 -1.57"/>
+  </joint>
+  <link name="camera_link">
+    <visual>
+      <origin xyz="0 0 0.0" rpy="0 0 0"/>
+      <geometry>
+        <box size="0.02 0.05 0.03"/>
+      </geometry>>
+    </visual>>
+  </link> -->
+<joint name="camera_tf_joint" type="fixed">
+    <parent link="camera_link"/>
+    <child link="camera_tf_link"/>
+    <origin xyz="0 0 0" rpy="-1.57 0 -1.57"/>
+  </joint>
+  <link name="camera_tf_link">
+  </link>
 </robot>
